File: A_REGISTER.kicad_sch (KiCad schematic)
At the start: 22 parts, among them U10 74LS173, U11 74LS173, U12 74LS245

Commit message: Some inverting signal commands are modified
Other:
- note added: "DB0~DB7 ==> DATA BUS 0 TO 7 ~{LOAD-A_REG} ==> FETCH THE DATA FROM BUS TO REGISTER CLK ==> CLOCK INPUT REG-A_Res ==> RESET THE CONTENT OF THE REGISTER ~{EN-A_REG} ==> OUTPUT THE DATA FROM REGISTER TO BUS"
- note removed: "DB0~DB7 ==> DATA BUS 0 TO 7 !LOAD-A_REG ==> FETCH THE DATA FROM BUS TO REGISTER CLK ==> CLOCK INPUT REG-A_Res ==> RESET THE CONTENT OF THE REGISTER !EN-A_REG ==> OUTPUT THE DATA FROM REGISTER TO BUS"
Changed lines of the file:
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@@
 		)
 	)
-	(text "DB0~DB7 ==> DATA BUS 0 TO 7\n!LOAD-A_REG ==> FETCH THE DATA FROM BUS TO REGISTER\nCLK ==> CLOCK INPUT\nREG-A_Res ==> RESET THE CONTENT OF THE REGISTER\n!EN-A_REG ==> OUTPUT THE DATA FROM REGISTER TO BUS"
+	(text "DB0~DB7 ==> DATA BUS 0 TO 7\n~{LOAD-A_REG} ==> FETCH THE DATA FROM BUS TO REGISTER\nCLK ==> CLOCK INPUT\nREG-A_Res ==> RESET THE CONTENT OF THE REGISTER\n~{EN-A_REG} ==> OUTPUT THE DATA FROM REGISTER TO BUS"
 		(exclude_from_sim no)
 		(at 43.18 56.642 0)
