File: B_REGISTER.kicad_sch (KiCad schematic)
At the start: 22 parts, among them U13 74LS173, U14 74LS173, U15 74LS245

Commit message: Some inverting signal commands are modified
Other:
- note added: "DB0~DB7 ==> DATA BUS 0 TO 7 ~{LOAD-B_REG} ==> FETCH THE DATA FROM BUS TO REGISTER CLK ==> CLOCK INPUT REG-B_Res ==> RESET THE CONTENT OF THE REGISTER ~{EN-B_REG} ==> OUTPUT THE DATA FROM REGISTER TO BUS"
- note removed: "DB0~DB7 ==> DATA BUS 0 TO 7 !LOAD-B_REG ==> FETCH THE DATA FROM BUS TO REGISTER CLK ==> CLOCK INPUT REG-B_Res ==> RESET THE CONTENT OF THE REGISTER !EN-B_REG ==> OUTPUT THE DATA FROM REGISTER TO BUS"
Changed lines of the file:
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@@
 		)
 	)
-	(text "DB0~DB7 ==> DATA BUS 0 TO 7\n!LOAD-B_REG ==> FETCH THE DATA FROM BUS TO REGISTER\nCLK ==> CLOCK INPUT\nREG-B_Res ==> RESET THE CONTENT OF THE REGISTER\n!EN-B_REG ==> OUTPUT THE DATA FROM REGISTER TO BUS"
+	(text "DB0~DB7 ==> DATA BUS 0 TO 7\n~{LOAD-B_REG} ==> FETCH THE DATA FROM BUS TO REGISTER\nCLK ==> CLOCK INPUT\nREG-B_Res ==> RESET THE CONTENT OF THE REGISTER\n~{EN-B_REG} ==> OUTPUT THE DATA FROM REGISTER TO BUS"
 		(exclude_from_sim no)
 		(at 40.64 56.642 0)
